File: pidroponic_uHAT/pidroponic_uHAT.sch (KiCad schematic (older format))
At the start: 28 parts, among them J1 GPIO_CONNECTOR, J2 1935161, J3 B4B-PH-K-S_LF__SN_, J4 B4B-PH-K-S_LF__SN_, J5 B4B-PH-K-S_LF__SN_, J6 B6B-PH-K-S_LF__SN_, J7 B4B-PH-K-S_LF__SN_, J8 TI ADS1115 Breakout, J9 B4B-PH-K-S_LF__SN_, Q1 DMG2305UX-13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

Commit message: updates over the last few evenings.
Parts:
- J2: footprint digikey-footprints:Terminal_Block_D1.3mm_P5mm -> TerminalBlock_Phoenix:TerminalBlock_Phoenix_PT-1,5-2-5.0-H_1x02_P5.00mm_Horizontal
Changed lines of the file:
@@
 F 0 "J2" V 625 5933 50  0000 C CNN
 F 1 "1935161" V 716 5933 50  0000 C CNN
-F 2 "digikey-footprints:Terminal_Block_D1.3mm_P5mm" H 1050 6050 60  0001 L CNN
+F 2 "TerminalBlock_Phoenix:TerminalBlock_Phoenix_PT-1,5-2-5.0-H_1x02_P5.00mm_Horizontal" H 1050 6050 60  0001 L CNN
 F 3 "https://media.digikey.com/pdf/Data%20Sheets/Phoenix%20Contact%20PDFs/1935161.pdf" H 1050 6150 60  0001 L CNN
 F 4 "277-1667-ND" H 1050 6250 60  0001 L CNN "Digi-Key_PN"

Commit message: Update to the uHAT, given learning new things.
* Removed the 5v linear regulator. Relays draw too much current for this to be safe. Off-board switching DC-DC buck converters are inexpensive up to 3A. Recommend using an LM2596 board.
* ADC pins configured for 3 thermistors (4.7k pullup through thermistor + filter cap) + one direct ADC feed for connecting a 3.3v analog PH Sensor
* Unified board design specs to make the 'fab' one the same as the 'homeproto'. We'll try traces this big with home proto and see where that gets us. In that vein, removed all but four vias.

General notes about this version:
* Soldering both sides of the header pins makes it possible to use those pads as vias, greatly reducing the number of 'fiddly things' you have to do.
* Removed the need for 16v 10uf caps, by dropping all the on-board voltages to 5v. Terminal block can be direct-wire soldered in place. No need for screw terminals if you don't want them.
Parts:
- removed J9: B4B-PH-K-S_LF__SN_, Connector_JST:JST_PH_B4B-PH-K_1x04_P2.00mm_Vertical, symbol dk_Rectangular-Connectors-Headers-Male-Pins:B4B-PH-K-S_LF__SN_
- removed U1: LM7805_TO220, Package_TO_SOT_THT:TO-220-3_Vertical, symbol Regulator_Linear:LM7805_TO220
- added C3, C4: 10uf, Capacitor_SMD:C_0805_2012Metric, symbol Device:C
- added J10: Therm 1, Connector_JST:JST_PH_B2B-PH-K_1x02_P2.00mm_Vertical, symbol dk_Rectangular-Connectors-Headers-Male-Pins:B2B-PH-K-S_LF__SN_
- added J11: Therm 2, Connector_JST:JST_PH_B2B-PH-K_1x02_P2.00mm_Vertical, symbol dk_Rectangular-Connectors-Headers-Male-Pins:B2B-PH-K-S_LF__SN_
- added J9: Analog PH, Connector_JST:JST_PH_B3B-PH-K_1x03_P2.00mm_Vertical, symbol dk_Rectangular-Connectors-Headers-Male-Pins:B3B-PH-K-S_LF__SN_
- added R10, R11, R12: 4.7k, Resistor_SMD:R_0805_2012Metric, symbol Device:R
- C1, C2: Description CAP CER 10UF 16V X5R 0805 -> CAP CER 10UF 10V X5R 0805; Digi-Key_PN 445-7644-1-ND -> 1276-1052-1-ND
- J3: value B4B-PH-K-S_LF__SN_ -> Prox 0
- J4: value B4B-PH-K-S_LF__SN_ -> Prox 1
- J5: value B4B-PH-K-S_LF__SN_ -> Prox 2
- J6: value B6B-PH-K-S_LF__SN_ -> 4 Chan Relay
- J7: value B4B-PH-K-S_LF__SN_ -> Therm 0; footprint Connector_JST:JST_PH_B4B-PH-K_1x04_P2.00mm_Vertical -> Connector_JST:JST_PH_B2B-PH-K_1x02_P2.00mm_Vertical; symbol dk_Rectangular-Connectors-Headers-Male-Pins:B4B-PH-K-S_LF__SN_ -> dk_Rectangular-Connectors-Headers-Male-Pins:B2B-PH-K-S_LF__SN_; Digi-Key_PN 455-1706-ND -> 455-1704-ND
- J8: value TI ADS1115 Breakout -> TI ADS1115 Breakout Board
Connections:
- net P12V is gone; now on net EXT5V: C1.1, J2.1
- net +3V3: now also J9.2, R10.1, R11.1, R12.1; no longer J1.17 (Pin_17), J7.1
- net A0: now also J9.3; no longer J7.2
- net A1: now also C2.1, J7.1, R10.2; no longer J7.3
- net A2: now also C3.1, J10.1, R11.2
- net A3: now also C4.1, J11.1, R12.2
- net GND: now also J7.2, C3.2, C4.2, J10.2, J11.2, J9.1; no longer J7.4
- net EXT5V: now reaches Q1.3 (D), Q2.6 (E)
- net EXT5V: no longer C2.1
- no-connect marks 16 -> 17
Other:
- note added: "External Power Source"
- note removed: "12v Power Source"
- moved on the sheet: J2, J8
